Commit message: Add tool exchanger and screwdriver joints with corresponding links in macro.m1013.white.xacro

File: dsr_description2/xacro/macro.m1013.white.xacro (robot description, xacro)
@@ -242,4 +242,56 @@
 			</visual>
 		</link>
+		<joint name="tool_exchanger_joint" type="fixed">
+			<parent link="link_6"/>
+			<child link="onrobot_tool_exchanger"/>
+			<origin xyz="0 0 0.050" rpy="0 0 0"/>
+		</joint>
+		<link name="onrobot_tool_exchanger">
+			<inertial>
+				<mass value="0.5"/>
+				<inertia ixx="0.5" ixy="0" ixz="0" iyy="0.5" iyz="0" izz="0.5" />
+			</inertial>
+			<visual>
+				<origin xyz="0 0 -0.025" rpy="0 0 0"/>
+				<geometry>
+				<cylinder radius="0.050" length="0.100"/>
+				</geometry>
+				<material name="Black">
+					<color rgba="0.0 0.0 0.0 1.0"/>
+				</material>
+			</visual>
+			<collision>
+				<origin xyz="0 0 -0.050" rpy="0 0 0"/>
+				<geometry>
+				<cylinder radius="0.050" length="0.100"/>
+				</geometry>
+			</collision>
+		</link>
+		<joint name="screwdriver_joint" type="fixed">
+			<parent link="onrobot_tool_exchanger"/>
+			<child link="screwdriver"/>
+			<origin xyz="0 -0.065 0" rpy="3.1416 0 3.1416"/>
+		</joint>
+		<link name="screwdriver">
+			<inertial>
+				<mass value="1.5"/>
+				<inertia ixx="0.5" ixy="0" ixz="0" iyy="0.5" iyz="0" izz="0.5" />
+			</inertial>
+			<visual>
+				<origin xyz="0 0 0" rpy="0 0 0"/>
+				<geometry>
+					<mesh filename="package://dsr_description2/meshes/screwdriver_simple.stl" scale="0.001 0.001 0.001"/>
+				</geometry>
+				<material name="Gray">
+					<color rgba="0.50 0.5 0.5 1.0"/>
+				</material>
+			</visual>
+			<collision>
+				<origin xyz="0 0 0" rpy="0 0 0"/>
+				<geometry>
+					<mesh filename="package://dsr_description2/meshes/screwdriver_simple.stl" scale="0.001 0.001 0.001"/>
+				</geometry>
+			</collision>
+		</link>
 		<xacro:dsr_transmission />
 		<xacro:dsr_gazebo namespace="${namespace}" />

Commit message: Add approximated screwdriver TCP

File: dsr_description2/xacro/macro.m1013.white.xacro (robot description, xacro)
@@ -294,4 +294,10 @@
 			</collision>
 		</link>
+    <link name="screwdriver_tcp"/>
+    <joint name="screwdriver_tcp_joint" type="fixed">
+      <parent link="screwdriver"/>
+      <child link="screwdriver_tcp"/>
+      <origin xyz="0 -0.084 -0.16" rpy="3.1416 0 0"/>
+    </joint>
 		<xacro:dsr_transmission />
 		<xacro:dsr_gazebo namespace="${namespace}" />
